File: HW/eagle/Gamepad/controller_v1.1B.brd (EAGLE design)
At the start: 109.2 x 81.3 mm, 21 parts, among them IC1 MCP23017SP

Commit message: First testable
Connections:
- net +5V renamed +3V3
Routing:
- net +3V3: track 116.8 -> 114.3 mm
Changed lines of the file:
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@@
 <wire x1="36.83" y1="57.15" x2="45.72" y2="57.15" width="1.27" layer="16"/>
-</signal>
-<signal name="+5V">
-<contactref element="RENC1" pad="C"/>
-<contactref element="IC1" pad="9"/>
-<contactref element="U$1" pad="VCC"/>
-<contactref element="WIRE" pad="2"/>
-<wire x1="45.72" y1="72.39" x2="45.72" y2="64.77" width="1.27" layer="16"/>
-<wire x1="45.72" y1="64.77" x2="48.26" y2="62.23" width="1.27" layer="16"/>
-<wire x1="48.26" y1="62.23" x2="48.26" y2="60.452" width="1.27" layer="16"/>
-<wire x1="48.26" y1="60.452" x2="48.26" y2="58.42" width="1.27" layer="16"/>
-<wire x1="48.26" y1="58.42" x2="53.34" y2="53.34" width="1.27" layer="16"/>
-<wire x1="53.34" y1="53.34" x2="53.34" y2="27.94" width="1.27" layer="16"/>
-<wire x1="52.07" y1="26.67" x2="50.8" y2="26.67" width="1.27" layer="16"/>
-<wire x1="53.34" y1="27.94" x2="52.07" y2="26.67" width="1.27" layer="16"/>
-<wire x1="46.99" y1="10.16" x2="40.64" y2="16.51" width="1.27" layer="16"/>
-<via x="40.64" y="16.51" extent="1-16" drill="0.6" diameter="1.27" shape="square"/>
-<wire x1="40.64" y1="16.51" x2="40.64" y2="26.67" width="1.27" layer="1"/>
-<via x="40.64" y="26.67" extent="1-16" drill="0.6" diameter="1.27" shape="square"/>
-<wire x1="40.64" y1="26.67" x2="50.8" y2="26.67" width="1.27" layer="16"/>
-<wire x1="46.99" y1="10.16" x2="59.69" y2="10.16" width="1.27" layer="16"/>
-<wire x1="59.69" y1="10.16" x2="59.69" y2="5.08" width="1.27" layer="16"/>
-<wire x1="59.69" y1="5.08" x2="77.47" y2="5.08" width="1.27" layer="16"/>
-<wire x1="77.47" y1="5.08" x2="77.47" y2="6.35" width="1.27" layer="16"/>
 </signal>
 <signal name="I2C_CLK">
@@
 <wire x1="64.77" y1="8.89" x2="64.77" y2="7.62" width="1.27" layer="16"/>
 </signal>
+<signal name="+3V3">
+<contactref element="WIRE" pad="2"/>
+<contactref element="IC1" pad="9"/>
+<contactref element="U$1" pad="VCC"/>
+<wire x1="45.72" y1="72.39" x2="45.72" y2="64.77" width="1.27" layer="16"/>
+<wire x1="45.72" y1="64.77" x2="48.26" y2="62.23" width="1.27" layer="16"/>
+<wire x1="48.26" y1="62.23" x2="48.26" y2="60.452" width="1.27" layer="16"/>
+<wire x1="48.26" y1="60.452" x2="48.26" y2="59.69" width="1.27" layer="16"/>
+<wire x1="48.26" y1="59.69" x2="53.34" y2="54.61" width="1.27" layer="16"/>
+<wire x1="53.34" y1="54.61" x2="53.34" y2="27.94" width="1.27" layer="16"/>
+<contactref element="RENC1" pad="C"/>
+<wire x1="53.34" y1="27.94" x2="52.07" y2="26.67" width="1.27" layer="16"/>
+<wire x1="52.07" y1="26.67" x2="50.8" y2="26.67" width="1.27" layer="16"/>
+<wire x1="50.8" y1="26.67" x2="41.91" y2="26.67" width="1.27" layer="16"/>
+<via x="41.91" y="26.67" extent="1-16" drill="0.6" shape="square"/>
+<wire x1="41.91" y1="26.67" x2="41.91" y2="16.51" width="1.27" layer="1"/>
+<via x="41.91" y="16.51" extent="1-16" drill="0.6" shape="square"/>
+<wire x1="41.91" y1="16.51" x2="41.91" y2="13.97" width="1.27" layer="16"/>
+<wire x1="41.91" y1="13.97" x2="45.72" y2="10.16" width="1.27" layer="16"/>
+<wire x1="45.72" y1="10.16" x2="58.42" y2="10.16" width="1.27" layer="16"/>
+<wire x1="58.42" y1="10.16" x2="59.69" y2="8.89" width="1.27" layer="16"/>
+<wire x1="59.69" y1="8.89" x2="59.69" y2="6.35" width="1.27" layer="16"/>
+<wire x1="59.69" y1="6.35" x2="60.96" y2="5.08" width="1.27" layer="16"/>
+<wire x1="60.96" y1="5.08" x2="77.47" y2="5.08" width="1.27" layer="16"/>
+<wire x1="77.47" y1="5.08" x2="77.47" y2="6.35" width="1.27" layer="16"/>
+</signal>
 </signals>
