File: HW/eagle/Gamepad/controller_v1.1B.sch (EAGLE design)
At the start: 21 parts, among them IC1 MCP23017SP

Commit message: First testable
Connections:
- net +5V renamed +3V3
Changed lines of the file:
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@@
 <part name="R3" library="eagle-ltspice" deviceset="R" device="0207/10" value="10k"/>
 <part name="R4" library="eagle-ltspice" deviceset="R" device="0207/10" value="10K"/>
-<part name="P+1" library="supply1" deviceset="+5V" device=""/>
-<part name="P+2" library="supply1" deviceset="+5V" device=""/>
-<part name="P+4" library="supply1" deviceset="+5V" device=""/>
 <part name="GND1" library="supply1" deviceset="GND" device=""/>
 <part name="GND2" library="supply1" deviceset="GND" device=""/>
 <part name="GND3" library="supply1" deviceset="GND" device=""/>
-<part name="P+5" library="supply1" deviceset="+5V" device=""/>
 <part name="GND4" library="supply1" deviceset="GND" device=""/>
 <part name="GND5" library="supply1" deviceset="GND" device=""/>
@@
 <part name="U$12" library="switch" deviceset="T_SW_RUBBER" device="2PIN"/>
 <part name="U$13" library="switch" deviceset="T_SW_RUBBER" device="2PIN"/>
+<part name="+3V1" library="supply1" deviceset="+3V3" device=""/>
+<part name="+3V2" library="supply1" deviceset="+3V3" device=""/>
+<part name="+3V3" library="supply1" deviceset="+3V3" device=""/>
+<part name="+3V4" library="supply1" deviceset="+3V3" device=""/>
 </parts>
 <sheets>
@@
 <instance part="R3" gate="G$1" x="-17.78" y="-22.86" rot="R270"/>
 <instance part="R4" gate="G$1" x="-10.16" y="-22.86" rot="R270"/>
-<instance part="P+1" gate="1" x="-20.32" y="-53.34" rot="R90"/>
-<instance part="P+2" gate="1" x="-22.86" y="20.32" rot="R90"/>
-<instance part="P+4" gate="1" x="-2.54" y="40.64" rot="R270"/>
 <instance part="GND1" gate="1" x="60.96" y="-66.04"/>
 <instance part="GND2" gate="1" x="-30.48" y="-66.04"/>
 <instance part="GND3" gate="1" x="27.94" y="35.56"/>
-<instance part="P+5" gate="1" x="15.24" y="38.1" rot="R90"/>
 <instance part="GND4" gate="1" x="-12.7" y="38.1"/>
 <instance part="GND5" gate="1" x="27.94" y="-66.04"/>
@@
 <instance part="U$12" gate="G$1" x="53.34" y="-48.26"/>
 <instance part="U$13" gate="G$1" x="53.34" y="-58.42"/>
+<instance part="+3V1" gate="G$1" x="-2.54" y="40.64" rot="R270"/>
+<instance part="+3V2" gate="G$1" x="-22.86" y="20.32" rot="R90"/>
+<instance part="+3V3" gate="G$1" x="15.24" y="38.1" rot="R90"/>
+<instance part="+3V4" gate="G$1" x="-20.32" y="-53.34" rot="R90"/>
 </instances>
 <busses>
@@
 </segment>
 </net>
-<net name="+5V" class="0">
-<segment>
-<pinref part="RENC1" gate="A" pin="C"/>
-<wire x1="-10.16" y1="-53.34" x2="-17.78" y2="-53.34" width="0.1524" layer="91"/>
-<pinref part="P+1" gate="1" pin="+5V"/>
-</segment>
-<segment>
-<pinref part="P+2" gate="1" pin="+5V"/>
-<pinref part="IC1" gate="G$1" pin="VDD"/>
-<wire x1="-20.32" y1="20.32" x2="7.62" y2="20.32" width="0.1524" layer="91"/>
-</segment>
-<segment>
-<wire x1="25.4" y1="50.8" x2="25.4" y2="38.1" width="0.1524" layer="91"/>
-<wire x1="25.4" y1="38.1" x2="17.78" y2="38.1" width="0.1524" layer="91"/>
-<pinref part="P+5" gate="1" pin="+5V"/>
-<pinref part="U$1" gate="G$1" pin="+5V"/>
-</segment>
-<segment>
-<pinref part="WIRE" gate="-2" pin="S"/>
-<pinref part="P+4" gate="1" pin="+5V"/>
-<wire x1="-17.78" y1="43.18" x2="-7.62" y2="43.18" width="0.1524" layer="91"/>
-<wire x1="-7.62" y1="43.18" x2="-7.62" y2="40.64" width="0.1524" layer="91"/>
-<wire x1="-7.62" y1="40.64" x2="-5.08" y2="40.64" width="0.1524" layer="91"/>
-</segment>
-</net>
 <net name="I2C_CLK" class="0">
 <segment>
@@
 </segment>
 </net>
+<net name="+3V3" class="0">
+<segment>
+<pinref part="WIRE" gate="-2" pin="S"/>
+<wire x1="-17.78" y1="43.18" x2="-7.62" y2="43.18" width="0.1524" layer="91"/>
+<wire x1="-7.62" y1="43.18" x2="-7.62" y2="40.64" width="0.1524" layer="91"/>
+<wire x1="-7.62" y1="40.64" x2="-5.08" y2="40.64" width="0.1524" layer="91"/>
+<pinref part="+3V1" gate="G$1" pin="+3V3"/>
+</segment>
+<segment>
+<pinref part="IC1" gate="G$1" pin="VDD"/>
+<wire x1="-20.32" y1="20.32" x2="7.62" y2="20.32" width="0.1524" layer="91"/>
+<pinref part="+3V2" gate="G$1" pin="+3V3"/>
+</segment>
+<segment>
+<wire x1="25.4" y1="50.8" x2="25.4" y2="38.1" width="0.1524" layer="91"/>
+<wire x1="25.4" y1="38.1" x2="17.78" y2="38.1" width="0.1524" layer="91"/>
+<pinref part="U$1" gate="G$1" pin="+5V"/>
+<pinref part="+3V3" gate="G$1" pin="+3V3"/>
+</segment>
+<segment>
+<pinref part="RENC1" gate="A" pin="C"/>
+<wire x1="-10.16" y1="-53.34" x2="-17.78" y2="-53.34" width="0.1524" layer="91"/>
+<pinref part="+3V4" gate="G$1" pin="+3V3"/>
+</segment>
+</net>
