File: HW/eagle/Port/Adapter_v1.1B.brd (EAGLE design)
At the start: 79 x 74.9 mm, 9 parts, among them X1 057-040-1, X2 057-010-1, X3 057-010-1, X4 057-010-1, X5 057-010-1, X6 22-23-2021, X7 22-23-2021

Commit message: First testable
Connections:
- removed net +12V: J1.1, X7.2
- removed net N$1: JP1.1, X1.2, X1.4
- new net +3V3: X1.1, X2.9, X3.9, X4.9, X5.9, X6.2
- net +5V: now also J1.1, JP1.1, X1.2, X1.4, X7.2; no longer X2.9, X3.9, X4.9, X5.9, X6.2
Routing:
- net +3V3: track 0.00 -> 127.9 mm, vias 0 -> 5
- net +5V: track 146.8 -> 58.5 mm, vias 4 -> 3
- net +12V: track 22.1 -> 0.00 mm, vias 1 -> 0
- net N$1: track 17.8 -> 0.00 mm, vias 2 -> 0
- net GND: track 320.5 -> 319.5 mm
Changed lines of the file:
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@@
 <wire x1="5.08" y1="35.56" x2="10.16" y2="35.56" width="1.27" layer="1"/>
 <via x="10.16" y="35.56" extent="1-16" drill="0.6" shape="square"/>
-<wire x1="5.08" y1="67.77" x2="6.88" y2="67.77" width="1.27" layer="1"/>
-<wire x1="6.88" y1="67.77" x2="9.88" y2="64.77" width="1.27" layer="1"/>
 <wire x1="58.42" y1="63.5" x2="58.42" y2="67.31" width="1.27" layer="1"/>
 <via x="58.42" y="67.31" extent="1-16" drill="0.6" shape="square"/>
@@
 <wire x1="25.4" y1="73.66" x2="13.97" y2="73.66" width="1.27" layer="16"/>
 <wire x1="13.97" y1="73.66" x2="10.16" y2="69.85" width="1.27" layer="16"/>
-<wire x1="10.16" y1="69.85" x2="10.16" y2="65.05" width="1.27" layer="16"/>
+<wire x1="10.16" y1="69.85" x2="10.16" y2="67.77" width="1.27" layer="16"/>
+<wire x1="10.16" y1="67.31" x2="10.16" y2="65.05" width="1.27" layer="16"/>
 <wire x1="10.16" y1="65.05" x2="9.88" y2="64.77" width="1.27" layer="16"/>
 <wire x1="26.67" y1="46.99" x2="25.4" y2="46.99" width="1.27" layer="16"/>
@@
 <wire x1="10.16" y1="40.64" x2="10.16" y2="64.49" width="1.27" layer="16"/>
 <wire x1="10.16" y1="64.49" x2="9.88" y2="64.77" width="1.27" layer="16"/>
+<wire x1="5.08" y1="67.77" x2="10.16" y2="67.77" width="1.27" layer="16"/>
+<wire x1="10.16" y1="67.77" x2="10.16" y2="67.31" width="1.27" layer="16"/>
 </signal>
 <signal name="+5V">
-<contactref element="X2" pad="9"/>
-<contactref element="X3" pad="9"/>
-<contactref element="X5" pad="9"/>
-<contactref element="X4" pad="9"/>
-<contactref element="X6" pad="2"/>
 <contactref element="JP1" pad="2"/>
-<wire x1="15.24" y1="69.85" x2="12.7" y2="67.31" width="1.27" layer="16"/>
-<wire x1="12.7" y1="67.31" x2="12.7" y2="58.42" width="1.27" layer="16"/>
-<wire x1="12.7" y1="58.42" x2="21.59" y2="49.53" width="1.27" layer="16"/>
-<wire x1="21.59" y1="49.53" x2="29.21" y2="49.53" width="1.27" layer="16"/>
-<wire x1="29.21" y1="49.53" x2="36.83" y2="49.53" width="1.27" layer="16"/>
-<wire x1="36.83" y1="49.53" x2="39.37" y2="46.99" width="1.27" layer="16"/>
-<wire x1="39.37" y1="46.99" x2="39.37" y2="36.83" width="1.27" layer="16"/>
-<wire x1="39.37" y1="36.83" x2="39.37" y2="24.13" width="1.27" layer="16"/>
-<wire x1="39.37" y1="13.97" x2="39.37" y2="10.16" width="1.27" layer="16"/>
-<wire x1="29.21" y1="46.99" x2="29.21" y2="49.53" width="1.27" layer="16"/>
-<wire x1="29.21" y1="24.13" x2="39.37" y2="24.13" width="1.27" layer="16"/>
-<wire x1="57.15" y1="13.97" x2="52.07" y2="13.97" width="1.27" layer="16"/>
-<via x="52.07" y="13.97" extent="1-16" drill="0.6" shape="square"/>
-<wire x1="52.07" y1="13.97" x2="39.37" y2="13.97" width="1.27" layer="1"/>
-<via x="39.37" y="13.97" extent="1-16" drill="0.6" shape="square"/>
-<wire x1="57.15" y1="36.83" x2="52.07" y2="36.83" width="1.27" layer="16"/>
-<via x="52.07" y="36.83" extent="1-16" drill="0.6" shape="square"/>
-<wire x1="52.07" y1="36.83" x2="39.37" y2="36.83" width="1.27" layer="1"/>
-<via x="39.37" y="36.83" extent="1-16" drill="0.6" shape="square"/>
-<wire x1="12.7" y1="40.64" x2="12.7" y2="58.42" width="1.27" layer="16"/>
-<wire x1="39.37" y1="24.13" x2="39.37" y2="13.97" width="1.27" layer="16"/>
+<contactref element="J1" pad="1"/>
+<contactref element="X7" pad="2"/>
+<wire x1="5.08" y1="61.67" x2="12.7" y2="61.67" width="1.27" layer="1"/>
+<wire x1="12.7" y1="61.67" x2="12.7" y2="62.23" width="1.27" layer="1"/>
+<via x="12.7" y="62.23" extent="1-16" drill="0.6" shape="square"/>
+<wire x1="12.7" y1="62.23" x2="12.7" y2="68.58" width="1.27" layer="16"/>
+<wire x1="12.7" y1="68.58" x2="13.97" y2="69.85" width="1.27" layer="16"/>
+<wire x1="13.97" y1="69.85" x2="15.24" y2="69.85" width="1.27" layer="16"/>
+<wire x1="5.08" y1="61.67" x2="5.08" y2="46.99" width="1.27" layer="16"/>
+<wire x1="5.08" y1="46.99" x2="7.62" y2="44.45" width="1.27" layer="16"/>
+<wire x1="7.62" y1="44.45" x2="7.62" y2="40.64" width="1.27" layer="16"/>
+<contactref element="X1" pad="4"/>
+<contactref element="X1" pad="2"/>
+<contactref element="JP1" pad="1"/>
+<wire x1="25.4" y1="63.5" x2="25.4" y2="67.31" width="1.27" layer="1"/>
+<via x="25.4" y="67.31" extent="1-16" drill="0.6" shape="square"/>
+<wire x1="25.4" y1="67.31" x2="22.86" y2="67.31" width="1.27" layer="16"/>
+<via x="22.86" y="67.31" extent="1-16" drill="0.6" shape="square"/>
+<wire x1="22.86" y1="67.31" x2="22.86" y2="63.5" width="1.27" layer="1"/>
+<wire x1="17.78" y1="69.85" x2="20.32" y2="69.85" width="1.27" layer="16"/>
+<wire x1="20.32" y1="69.85" x2="22.86" y2="67.31" width="1.27" layer="16"/>
+<wire x1="15.24" y1="69.85" x2="17.78" y2="69.85" width="0.6096" layer="16"/>
 </signal>
 <signal name="I2C-CLK">
@@
 <wire x1="44.45" y1="21.59" x2="44.45" y2="16.51" width="1.27" layer="16"/>
 </signal>
-<signal name="N$1">
-<contactref element="X1" pad="2"/>
-<contactref element="X1" pad="4"/>
-<contactref element="JP1" pad="1"/>
-<wire x1="25.4" y1="63.5" x2="25.4" y2="67.31" width="1.27" layer="1"/>
-<via x="25.4" y="67.31" extent="1-16" drill="0.6" shape="square"/>
-<wire x1="25.4" y1="67.31" x2="22.86" y2="67.31" width="1.27" layer="16"/>
-<wire x1="22.86" y1="63.5" x2="22.86" y2="67.31" width="1.27" layer="1"/>
-<via x="22.86" y="67.31" extent="1-16" drill="0.6" shape="square"/>
-<wire x1="22.86" y1="67.31" x2="22.86" y2="69.85" width="1.27" layer="16"/>
-<wire x1="22.86" y1="69.85" x2="17.78" y2="69.85" width="1.27" layer="16"/>
-</signal>
-<signal name="+12V">
-<contactref element="X7" pad="2"/>
-<contactref element="J1" pad="1"/>
-<wire x1="7.62" y1="40.64" x2="7.62" y2="53.34" width="1.27" layer="16"/>
-<wire x1="7.62" y1="53.34" x2="5.08" y2="55.88" width="1.27" layer="16"/>
-<via x="5.08" y="55.88" extent="1-16" drill="0.6" shape="square"/>
-<wire x1="5.08" y1="55.88" x2="5.08" y2="61.67" width="1.27" layer="1"/>
+<signal name="+3V3">
+<contactref element="X1" pad="1"/>
+<contactref element="X6" pad="2"/>
+<contactref element="X2" pad="9"/>
+<contactref element="X3" pad="9"/>
+<contactref element="X4" pad="9"/>
+<contactref element="X5" pad="9"/>
+<wire x1="12.7" y1="40.64" x2="13.97" y2="40.64" width="1.27" layer="16"/>
+<wire x1="13.97" y1="40.64" x2="22.86" y2="49.53" width="1.27" layer="16"/>
+<wire x1="22.86" y1="49.53" x2="29.21" y2="49.53" width="1.27" layer="16"/>
+<wire x1="29.21" y1="49.53" x2="36.83" y2="49.53" width="1.27" layer="16"/>
+<wire x1="36.83" y1="49.53" x2="39.37" y2="46.99" width="1.27" layer="16"/>
+<wire x1="39.37" y1="46.99" x2="39.37" y2="36.83" width="1.27" layer="16"/>
+<wire x1="39.37" y1="36.83" x2="39.37" y2="24.13" width="1.27" layer="16"/>
+<wire x1="39.37" y1="24.13" x2="39.37" y2="15.24" width="1.27" layer="16"/>
+<wire x1="39.37" y1="13.97" x2="39.37" y2="10.16" width="1.27" layer="16"/>
+<wire x1="22.86" y1="60.96" x2="22.86" y2="57.15" width="1.27" layer="1"/>
+<via x="22.86" y="57.15" extent="1-16" drill="0.6" shape="square"/>
+<wire x1="22.86" y1="57.15" x2="22.86" y2="49.53" width="1.27" layer="16"/>
+<wire x1="29.21" y1="46.99" x2="29.21" y2="49.53" width="1.27" layer="16"/>
+<wire x1="29.21" y1="24.13" x2="39.37" y2="24.13" width="1.27" layer="16"/>
+<wire x1="57.15" y1="36.83" x2="52.07" y2="36.83" width="1.27" layer="16"/>
+<via x="52.07" y="36.83" extent="1-16" drill="0.6" shape="square"/>
+<wire x1="52.07" y1="36.83" x2="39.37" y2="36.83" width="1.27" layer="1"/>
+<via x="39.37" y="36.83" extent="1-16" drill="0.6" shape="square"/>
+<wire x1="57.15" y1="13.97" x2="52.07" y2="13.97" width="1.27" layer="16"/>
+<via x="52.07" y="13.97" extent="1-16" drill="0.6" shape="square"/>
+<wire x1="52.07" y1="13.97" x2="39.37" y2="13.97" width="1.27" layer="1"/>
+<via x="39.37" y="13.97" extent="1-16" drill="0.6" shape="square"/>
+<wire x1="39.37" y1="13.97" x2="39.37" y2="15.24" width="1.27" layer="16"/>
 </signal>
 </signals>
